File: schematic/rs232RGBLEDController.sch (EAGLE design)
At the start: 41 parts, among them IC1 WS2811-SOP8, J1 AVR_SPI_PRG_62X3_LOCK, Q4 MOSFET-NCHANNELBSS123LT1G, U1 V_REG_LDOSMD, U3 ATMEGA8A-AU-TQFP32, X1 CRYSTALS-NOGND-HC49

Commit message: Minor.
Parts:
- U$2: SPICEPREFIX (none) -> B
Other:
- moved on the sheet: C1, C2, C3, C4, C5, C6, C7, C8, C9, D1, D2, F1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
